File: KI_Osciloscopio/Osciloscopio.kicad_pcb (KiCad board)
At the start: 2 copper layers, 100 x 77 mm, 41 parts, among them CN1 Conector IZQ, CN2 Conector DER, J1 VIN, J2 Conn_Coaxial, J3 DISPLAY, J4 USB_B, U1 MCP6004, U2 74HC4051, U4 LM1117-3.3, U5 M95128

Commit message: Kicad Terminado
Parts:
- R1, R10, R11, R12, R13, R14, R15, R16, R17, R18, R19, R2, R20, R3, R4, R5, R6, R7, R9: footprint Resistor_THT:R_Axial_DIN0207_L6.3mm_D2.5mm_P7.62mm_Horizontal -> Resistor_THT:R_Axial_DIN0207_L6.3mm_D2.5mm_P10.16mm_Horizontal
- moved R13 4.14 mm to (68.6, 66.9)
- moved R15 2.88 mm to (61.0, 53.1)
- moved R14 2.80 mm to (57.2, 53.2)
- moved R16 2.03 mm to (71.4, 53.9)
- moved R17 2.02 mm to (75.0, 53.9)
- moved R6 1.77 mm to (77.6, 77.5)
- moved R9 1.44 mm to (73.0, 77.5)
- moved R4 1.43 mm to (93.2, 77.5)
- moved R3 1.43 mm to (89.4, 77.5)
- moved R5 1.42 mm to (81.8, 77.5)
- moved R1 1.12 mm to (96.8, 67.3)
- moved R2 1.12 mm to (85.5, 67.3)
Routing:
- net Net-(R1-Pad1): track 53.0 -> 57.8 mm
- net Net-(C12-Pad2): track 18.8 -> 22.8 mm
- net Net-(R16-Pad1): track 28.2 -> 31.6 mm
- net Net-(R13-Pad2): track 30.3 -> 33.6 mm
- net /A0: track 38.6 -> 36.1 mm
- net Net-(R2-Pad2): track 27.3 -> 25.6 mm
- net Net-(R3-Pad1): track 28.0 -> 26.5 mm
- net Net-(R4-Pad1): track 29.0 -> 27.5 mm
- net Net-(R9-Pad1): track 5.69 -> 4.17 mm
- net Net-(C11-Pad2): track 12.1 -> 13.5 mm
- net Net-(R10-Pad1): track 12.0 -> 10.7 mm
- net Net-(R5-Pad1): track 25.4 -> 24.2 mm
- net Net-(R6-Pad1): track 5.20 -> 4.14 mm
- net Net-(C1-Pad1): track 5.00 -> 5.59 mm
