File: KI_Osciloscopio/Osciloscopio.kicad_sch (KiCad schematic)
At the start: 46 parts, among them CN1 Conector IZQ, CN2 Conector DER, J1 Barrel Jack, J2 Conn_Coaxial, J3 OLED 128x64, J4 USB_B, U1 MCP6004, U2 74HC4051, U3 LM2940CT-5.0/NOPB, U4 LM1117-3.3, U5 M95128

Commit message: Cambie el circuito de alimentacion
Parts:
- removed C2: 1000uF, Capacitor_THT:C_Disc_D5.0mm_W2.5mm_P2.50mm, symbol Device:C
- removed C3, C4, C5: 100nF, Capacitor_THT:C_Disc_D5.0mm_W2.5mm_P2.50mm, symbol Device:C
- removed D3, D5: 1N4007, Diode_THT:D_DO-41_SOD81_P10.16mm_Horizontal, symbol Diode:1N4007
- removed D4: P6KE13A, Diode_THT:D_DO-15_P10.16mm_Horizontal, symbol Device:D_Schottky
- removed J1: Barrel Jack, Connector_BarrelJack:BarrelJack_Horizontal, symbol Connector:Barrel_Jack_Switch
- removed U3: LM2940CT-5.0/NOPB, Package_TO_SOT_THT:TO-220-3_Vertical, symbol AOI-LM2940CT:LM2940CT-5.0/NOPB
Connections:
- net Earth: no longer C6.2, C7.2, C8.2, C9.2, U4.1 (GND)
- new net: C6.2, C7.2, C8.2, C9.2, U4.1 (GND)
Other:
- moved on the sheet: C1, C11, C12, C6, C7, C8, C9, CN1, CN2, D6, J2, J3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

Commit message: Termine PCB
Parts:
- removed JP1: Jumper_2_Open, symbol Jumper:Jumper_2_Open
- added J1: VIN, Connector_PinHeader_2.54mm:PinHeader_1x01_P2.54mm_Vertical, symbol Connector:Conn_01x01_Male
- added unit 4 of U1
- J3: value OLED 128x64 -> DISPLAY; footprint (none) -> Connector_PinHeader_2.54mm:PinHeader_1x04_P2.54mm_Vertical
- J4: footprint Connector_USB:USB_B_Amphenol_MUSB-D511_Vertical_Rugged -> Connector_USB:USB_B_OST_USB-B1HSxx_Horizontal
- U4: footprint Package_TO_SOT_THT:TO-220-3_Vertical -> Package_TO_SOT_THT:TO-220-3_Horizontal_TabDown
Connections:
- net VBUS is gone; now on net VIN: J4.1 (VBUS)
- net 3.3V: now also CN2.20 (Pin_20), CN2.22 (Pin_22), J3.4 (Pin_4); no longer CN1.15 (Pin_15), CN1.16 (Pin_16), J3.3 (Pin_3)
- net A0: no longer CN1.38 (Pin_38)
- net A1: no longer CN1.36 (Pin_36)
- net CS: now also CN1.3 (Pin_3); no longer CN2.17 (Pin_17), CN2.18 (Pin_18)
- net D+: now also CN2.11 (Pin_11)
- net D-: now also CN2.13 (Pin_13)
- net D0: now also U2.6 (~{E}); no longer CN2.37 (Pin_37)
- net D1: now also U2.9 (S2); no longer CN2.35 (Pin_35)
- net D2: now also U2.10 (S1); no longer CN2.33 (Pin_33)
- net D3: now also U2.11 (S0); no longer CN2.31 (Pin_31)
- net D4: no longer CN2.29 (Pin_29)
- net D5: no longer CN2.27 (Pin_27)
- net D7: no longer CN2.23 (Pin_23), U2.10 (S1)
- net MISO: now also CN1.1 (Pin_1); no longer CN2.13 (Pin_13), CN2.14 (Pin_14)
- net MOSI: now also CN1.4 (Pin_4); no longer CN2.15 (Pin_15), CN2.16 (Pin_16)
- net SCK: now also CN1.2 (Pin_2); no longer CN2.11 (Pin_11), CN2.12 (Pin_12)
- net SCL: no longer CN2.3 (Pin_3)
- net SDA: no longer CN2.5 (Pin_5)
- net VIN: now also C6.1, D6.2 (A), J1.1 (Pin_1); no longer CN1.23 (Pin_23), CN1.24 (Pin_24)
- net GND: now reaches C6.2, C7.2, C8.2, C9.2, U4.1 (GND)
- net GND: now also C11.1, CN1.19 (Pin_19), CN1.20 (Pin_20), CN1.21 (Pin_21), CN1.7 (Pin_7), CN2.10 (Pin_10), CN2.19 (Pin_19), J2.2 (Ext), J3.3 (Pin_3), J4.4 (GND), J4.5 (Shield), R12.2, R17.2, R20.2, U1.11 (V-), U2.7 (VEE), U2.8 (GND), U5.4 (VSS)
- net A2: no longer names the net of CN1.31 (Pin_31)
- net A2: no longer CN1.34 (Pin_34)
- net A3: no longer names the net of CN1.32 (Pin_32)
- net A3: no longer CN1.33 (Pin_33)
- net A4: no longer names the net of CN1.30 (Pin_30)
- net A4: no longer CN1.35 (Pin_35)
- net A5: no longer names the net of CN1.28 (Pin_28)
- net A5: no longer CN1.37 (Pin_37)
- net AVDD: no longer names the net of CN2.7 (Pin_7)
- net AVDD: no longer CN2.8 (Pin_8)
- net BOOT0: no longer names the net of CN1.8 (Pin_8)
- net BOOT0: no longer CN1.7 (Pin_7)
- removed net D6: CN2.25 (Pin_25), CN2.26 (Pin_26), U2.9 (S2)
- removed net D8: CN2.21 (Pin_21), CN2.22 (Pin_22), U2.11 (S0)
- removed net D9: CN2.19 (Pin_19), CN2.20 (Pin_20), U2.6 (~{E})
- removed net Earth: C11.1, CN1.19 (Pin_19), CN1.20 (Pin_20), CN1.21 (Pin_21), CN1.22 (Pin_22), CN2.10 (Pin_10), CN2.9 (Pin_9), J2.2 (Ext), J3.4 (Pin_4), J4.4 (GND), J4.5 (Shield), R12.2, R17.2, R20.2, U1.11 (V-), U2.7 (VEE), U2.8 (GND), U5.4 (VSS)
- net IOREF: no longer names the net of CN1.11 (Pin_11)
- net IOREF: no longer CN1.12 (Pin_12)
- net NC: no longer names the net of CN1.10 (Pin_10)
- net NC: no longer CN1.9 (Pin_9)
- net NC2: no longer names the net of CN1.25 (Pin_25)
- net NC2: no longer CN1.26 (Pin_26)
- net NRST: no longer names the net of CN1.13 (Pin_13)
- net NRST: no longer CN1.14 (Pin_14)
- removed net PC10: CN1.1 (Pin_1), CN1.2 (Pin_2)
- removed net PC12: CN1.3 (Pin_3), CN1.4 (Pin_4)
- net PC9: no longer names the net of CN2.1 (Pin_1)
- net PC9: no longer CN2.2 (Pin_2)
- removed net VCC: C6.1, CN1.17 (Pin_17), CN1.18 (Pin_18), D6.2 (A)
- net VDD: no longer names the net of CN1.5 (Pin_5)
- net VDDD: no longer names the net of CN1.6 (Pin_6)
- no-connect marks 0 -> 57
Other:
- note removed: "ALIMENTACION"
- note removed: "VER LA PATA VDD DE LA TIRA DE PINES COINCIDE CON UNA LABEL DE LA FUENTE CREO QUE HAY QUE CAMBIAR EL NOMBRE"
- moved on the sheet: C6, C7, C8, C9, CN1, CN2, D6, J4, U4

Commit message: Plaquita
Parts:
- added H1, H2, H3, H4: MountingHole, MountingHole:MountingHole_2.5mm, symbol Mechanical:MountingHole
- U4: footprint Package_TO_SOT_THT:TO-220-3_Horizontal_TabDown -> Package_TO_SOT_THT:TO-220-3_Vertical
Changed lines of the file:
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@@
+    )
+  )
+  (symbol (lib_id "Mechanical:MountingHole") (at 182.88 128.27 0) (unit 1)
+    (in_bom yes) (on_board yes)
+    (property "Reference" "H3" (id 0) (at 185.42 126.9999 0)
+      (effects (font (size 1.27 1.27)) (justify left))
+    )
+    (property "Value" "MountingHole" (id 1) (at 185.42 129.5399 0)
+      (effects (font (size 1.27 1.27)) (justify left))
+    )
+    (property "Footprint" "MountingHole:MountingHole_2.5mm" (id 2) (at 182.88 128.27 0)
+      (effects (font (size 1.27 1.27)) hide)
+    )
+    (property "Datasheet" "~" (id 3) (at 182.88 128.27 0)
+      (effects (font (size 1.27 1.27)) hide)
     )
   )
@@
     (property "Reference" "U4" (id 0) (at 50.8 120.65 0))
     (property "Value" "LM1117-3.3" (id 1) (at 50.8 123.19 0))
-    (property "Footprint" "Package_TO_SOT_THT:TO-220-3_Horizontal_TabDown" (id 2) (at 50.8 127 0)
+    (property "Footprint" "Package_TO_SOT_THT:TO-220-3_Vertical" (id 2) (at 50.8 127 0)
       (effects (font (size 1.27 1.27)) hide)
     )
@@
     )
     (pin "1")
+  )
+  (symbol (lib_id "Mechanical:MountingHole") (at 182.88 113.03 0) (unit 1)
+    (in_bom yes) (on_board yes) (fields_autoplaced)
+    (property "Reference" "H1" (id 0) (at 185.42 111.7599 0)
+      (effects (font (size 1.27 1.27)) (justify left))
+    )
+    (property "Value" "MountingHole" (id 1) (at 185.42 114.2999 0)
+      (effects (font (size 1.27 1.27)) (justify left))
+    )
+    (property "Footprint" "MountingHole:MountingHole_2.5mm" (id 2) (at 182.88 113.03 0)
+      (effects (font (size 1.27 1.27)) hide)
+    )
+    (property "Datasheet" "~" (id 3) (at 182.88 113.03 0)
+      (effects (font (size 1.27 1.27)) hide)
+    )
+  )
+  (symbol (lib_id "Mechanical:MountingHole") (at 182.88 135.89 0) (unit 1)
+    (in_bom yes) (on_board yes)
+    (property "Reference" "H4" (id 0) (at 185.42 134.6199 0)
+      (effects (font (size 1.27 1.27)) (justify left))
+    )
+    (property "Value" "MountingHole" (id 1) (at 185.42 137.1599 0)
+      (effects (font (size 1.27 1.27)) (justify left))
+    )
+    (property "Footprint" "MountingHole:MountingHole_2.5mm" (id 2) (at 182.88 135.89 0)
+      (effects (font (size 1.27 1.27)) hide)
+    )
+    (property "Datasheet" "~" (id 3) (at 182.88 135.89 0)
+      (effects (font (size 1.27 1.27)) hide)
+    )
   )
   (symbol (lib_id "power:GND") (at 207.01 66.04 90) (unit 1)
@@
     )
     (pin "1")
+  )
+  (symbol (lib_id "Mechanical:MountingHole") (at 182.88 120.65 0) (unit 1)
+    (in_bom yes) (on_board yes) (fields_autoplaced)
+    (property "Reference" "H2" (id 0) (at 185.42 119.3799 0)
+      (effects (font (size 1.27 1.27)) (justify left))
+    )
+    (property "Value" "MountingHole" (id 1) (at 185.42 121.9199 0)
+      (effects (font (size 1.27 1.27)) (justify left))
+    )
+    (property "Footprint" "MountingHole:MountingHole_2.5mm" (id 2) (at 182.88 120.65 0)
+      (effects (font (size 1.27 1.27)) hide)
+    )
+    (property "Datasheet" "~" (id 3) (at 182.88 120.65 0)
+      (effects (font (size 1.27 1.27)) hide)
+    )
   )
   (symbol (lib_id "Connector_Generic:Conn_02x19_Odd_Even") (at 236.22 64.77 0) (mirror y) (unit 1)
@@
       (reference "D6") (unit 1) (value "1N5819") (footprint "Diode_THT:D_DO-41_SOD81_P10.16mm_Horizontal")
     )
+    (path "/75d3ff0f-115c-4378-9b81-fd0f11ad05fe"
+      (reference "H1") (unit 1) (value "MountingHole") (footprint "MountingHole:MountingHole_2.5mm")
+    )
+    (path "/e99fbe20-806a-40e1-9bf8-bdffbae677f9"
+      (reference "H2") (unit 1) (value "MountingHole") (footprint "MountingHole:MountingHole_2.5mm")
+    )
+    (path "/00f2927e-e587-4e7a-84f9-a5cfc7c92328"
+      (reference "H3") (unit 1) (value "MountingHole") (footprint "MountingHole:MountingHole_2.5mm")
+    )
+    (path "/77ef6575-0a27-443b-8cb7-30f11ffb647d"
+      (reference "H4") (unit 1) (value "MountingHole") (footprint "MountingHole:MountingHole_2.5mm")
+    )
     (path "/74b90397-90d9-4bb6-8803-5bafb712db5e"
       (reference "J1") (unit 1) (value "VIN") (footprint "Connector_PinHeader_2.54mm:PinHeader_1x01_P2.54mm_Vertical")
@@
     )
     (path "/3a131e3e-9f8a-40a2-8ed5-4e47ca92d0c5"
-      (reference "U4") (unit 1) (value "LM1117-3.3") (footprint "Package_TO_SOT_THT:TO-220-3_Horizontal_TabDown")
+      (reference "U4") (unit 1) (value "LM1117-3.3") (footprint "Package_TO_SOT_THT:TO-220-3_Vertical")
     )
     (path "/a42d33e8-de2f-46db-a677-30067a2a34ea"

Commit message: Kicad Terminado
Parts:
- R1, R10, R11, R12, R13, R14, R15, R16, R17, R18, R19, R2, R20, R3, R4, R5, R6, R7, R9: footprint Resistor_THT:R_Axial_DIN0207_L6.3mm_D2.5mm_P7.62mm_Horizontal -> Resistor_THT:R_Axial_DIN0207_L6.3mm_D2.5mm_P10.16mm_Horizontal
